Commit message: Mvoing Correctly

File: ros2_ur5_interface/models/desk.urdf.xacro (robot description, xacro)
@@ -1,10 +1,9 @@
 <?xml version="1.0" ?>
 <robot name="desk" xmlns:xacro="http://www.ros.org/wiki/xacro">
-  <!-- Static property -->
   <link name="desk">
     <!-- Inertial -->
     <inertial>
       <origin xyz="0.5 0.4 0.435" rpy="0 0 0" />
-      <mass value="10" />
+      <mass value="10000" />
       <inertia ixx="0.1" ixy="0" ixz="0" iyy="0.1" iyz="0" izz="0.1" />
     </inertial>

Commit message: Image Processing, Object Processing, Detection Adjustment, Obtaining Position and Orientation

File: ros2_ur5_interface/models/desk.urdf.xacro (robot description, xacro)
@@ -2,9 +2,10 @@
 <robot name="desk" xmlns:xacro="http://www.ros.org/wiki/xacro">
   <link name="desk">
+    <static>true</static>
     <!-- Inertial -->
     <inertial>
       <origin xyz="0.5 0.4 0.435" rpy="0 0 0" />
-      <mass value="10000" />
-      <inertia ixx="0.1" ixy="0" ixz="0" iyy="0.1" iyz="0" izz="0.1" />
+      <mass value="100000" />
+      <inertia ixx="1000000" ixy="0" ixz="0" iyy="1000000" iyz="0" izz="1000000" />
     </inertial>
     <!-- Base collision -->
