Commit message: Conversion Integration

File: ros2_ur5_interface/models/soft_robotics_gripper.xacro (robot description, xacro)
@@ -64,5 +64,5 @@
       <parent link="${prefix}soft_robotics_gripper_base_link" />
       <child link="${prefix}soft_robotics_right_finger_link1" />
-      <limit effort="1" velocity="1" lower="-0.35" upper="0.35" />
+      <limit effort="1" velocity="1" lower="-1" upper="1" />
       <axis xyz="1 0 0"/>
     </joint>

Commit message: Final Push

File: ros2_ur5_interface/models/soft_robotics_gripper.xacro (robot description, xacro)
@@ -7,9 +7,13 @@
     <color rgba="0 0 1 1" />
   </material>
-  <xacro:macro name="soft_robotics_gripper" params="prefix parent *origin">
-    <joint name="${prefix}soft_robotics_gripper_base_joint" type="fixed">
-      <origin xyz="0 0 0" rpy="0 0 0" />
+ <xacro:property name="rotation_z" value="$(arg rotation_z)"/>
+ <!-- Add a comment to indicate the value being passed -->
+ <!-- Rotation Z value: $(rotation_z) -->
+  <xacro:macro name="soft_robotics_gripper" params="prefix parent *origin rotation_z">
+    <joint name="${prefix}soft_robotics_gripper_base_joint" type="revolute">
+      <origin xyz="0 0 0" rpy="0 0 ${rotation_z}" />
       <parent link="${parent}" />
       <child link="${prefix}soft_robotics_gripper_base_link" />
+      <limit effort="1" velocity="1" lower="-3.14" upper="3.14" />
     </joint>
     <link name="${prefix}soft_robotics_gripper_base_link">
@@ -152,4 +156,17 @@
           <plugin>gz_ros2_control/GazeboSimSystem</plugin>
         </hardware>
+        <joint name="${prefix}soft_robotics_gripper_base_joint">
+          <command_interface name="position"/>
+          <command_interface name="velocity"/>
+          <state_interface name="position">
+            <param name="initial_value">0.0</param>
+          </state_interface>
+          <state_interface name="velocity">
+            <param name="initial_value">0.0</param>
+          </state_interface>
+          <state_interface name="effort">
+            <param name="initial_value">0.0</param>
+          </state_interface>
+        </joint>
         <joint name="${prefix}soft_robotics_gripper_left_finger_joint1">
           <command_interface name="position"/>
@@ -182,4 +199,13 @@
     </ros2_control>
     <!-- TRANSMISSION -->
+    <transmission name="${prefix}base_trans">
+      <type>transmission_interface/SimpleTransmission</type>
+      <joint name="${prefix}soft_robotics_gripper_base_joint">
+        <hardwareInterface>hardware_interface/PositionJointInterface</hardwareInterface>
+      </joint>
+      <actuator name="${prefix}base_motor">
+        <mechanicalReduction>1</mechanicalReduction>
+      </actuator>
+    </transmission>
     <transmission name="${prefix}right_finger_trans">
       <type>transmission_interface/SimpleTransmission</type>

File: ros2_ur5_interface/models/ur_gz.urdf.xacro (robot description, xacro)
@@ -48,4 +48,5 @@
      parent="tool0"
      prefix=""
+     rotation_z="$(arg rotation_z)"
      >
      <origin xyz="0 0 0" rpy="0 0 0" />          <!-- position robot in the desk -->
